File: vesc_mms_board/usb.kicad_sch (KiCad schematic)
At the start: 14 parts, among them J6 Conn_01x05, U1 CH334R, Y1 12Mhz

Commit message: pcb created
Parts:
- renumbered C2 to C3, C3 to C4, J6 to J4, R4 to R10, R5 to R11, R6 to R12, R8 to R13, R9 to R14, R3 to R9
Connections:
- net USB_DOWNSTREM_D+ is gone; now on net USB_DOWNSTREAM_D+: R12.1
- net USB_DOWNSTREM_D- is gone; now on net USB_DOWNSTREAM_D-: R11.2

Commit message: cehnaged leyour added vias
Parts:
- C4: footprint Capacitor_SMD:C_0603_1608Metric -> Capacitor_SMD:C_0402_1005Metric
Changed lines of the file:
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@@
 			)
 		)
-		(property "Footprint" "Capacitor_SMD:C_0603_1608Metric"
+		(property "Footprint" "Capacitor_SMD:C_0402_1005Metric"
 			(at 133.6548 74.93 0)
 			(effects

Commit message: Update rev 2.0, added step files
Parts:
- J4: footprint Connector_PinHeader_2.54mm:PinHeader_1x05_P2.54mm_Vertical -> Connector_JST:JST_XH_B5B-XH-A_1x05_P2.50mm_Vertical
Connections:
- net +5V: now also J4.5 (Pin_5); no longer J4.1 (Pin_1)
- net GND: now also J4.1 (Pin_1), J4.2 (Pin_2); no longer J4.4 (Pin_4), J4.5 (Pin_5)
- net USB_VESC_D-: now also J4.4 (Pin_4); no longer J4.2 (Pin_2)
Changed lines of the file:
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@@
 		(lib_id "Connector_Generic:Conn_01x05")
 		(at 226.06 68.58 0)
+		(mirror x)
 		(unit 1)
 		(exclude_from_sim no)
@@
 		(on_board yes)
 		(dnp no)
-		(fields_autoplaced yes)
 		(property "Reference" "J4"
-			(at 228.6 67.3099 0)
+			(at 228.6 69.8501 0)
 			(effects
 				(font
@@
 		)
 		(property "Value" "Conn_01x05"
-			(at 228.6 69.8499 0)
+			(at 228.6 67.3101 0)
 			(effects
 				(font
@@
 			)
 		)
-		(property "Footprint" "Connector_PinHeader_2.54mm:PinHeader_1x05_P2.54mm_Vertical"
+		(property "Footprint" "Connector_JST:JST_XH_B5B-XH-A_1x05_P2.50mm_Vertical"
 			(at 226.06 68.58 0)
 			(effects
