File: vesc_mms_board/vesc_mms_board.kicad_sch (KiCad schematic)
At the start: 8 parts

Commit message: pcb created
Parts:
- renumbered H3 to H1, H4 to H2, H5 to H3, H6 to H4, H7 to H5, H8 to H6, H9 to H7, H10 to H8

Commit message: fianl
Parts:
- H1, H2, H4, H7: footprint MountingHole:MountingHole_3.5mm -> MountingHole:MountingHole_4.3mm_M4
Other:
- moved on the sheet: H1, H2, H3, H4, H5, H6, H7

Commit message: updarte readme final desing rev a
Other:
- company: (none) -> Modu System
- title: (none) -> Flipsky MMS module 
Changed lines of the file:
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@@
 	(generator_version "8.0")
 	(paper "A4")
+	(title_block
+		(title "Flipsky MMS module ")
+		(date "2024-12-14")
+		(rev "A")
+		(company "Modu System")
+	)
 	(rectangle
 		(start 30.48 168.91)

Commit message: Update rev 2.0, added step files
Parts:
- removed H1: MountingHole, MountingHole:MountingHole_4.3mm_M4, symbol Mechanical:MountingHole
Changed lines of the file:
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@@
-	(symbol
-		(lib_id "Mechanical:MountingHole")
-		(at 46.99 184.15 0)
-		(unit 1)
-		(exclude_from_sim yes)
-		(in_bom no)
-		(on_board yes)
-		(dnp no)
-		(fields_autoplaced yes)
-		(property "Reference" "H1"
-			(at 49.53 182.8799 0)
-			(effects
-				(font
-					(size 1.27 1.27)
-				)
-				(justify left)
-			)
-		)
-		(property "Value" "MountingHole"
-			(at 49.53 185.4199 0)
-			(effects
-				(font
-					(size 1.27 1.27)
-				)
-				(justify left)
-				(hide yes)
-			)
-		)
-		(property "Footprint" "MountingHole:MountingHole_4.3mm_M4"
-			(at 46.99 184.15 0)
-			(effects
-				(font
-					(size 1.27 1.27)
-				)
-				(hide yes)
-			)
-		)
-		(property "Datasheet" "~"
-			(at 46.99 184.15 0)
-			(effects
-				(font
-					(size 1.27 1.27)
-				)
-				(hide yes)
-			)
-		)
-		(property "Description" "Mounting Hole without connection"
-			(at 46.99 184.15 0)
-			(effects
-				(font
-					(size 1.27 1.27)
-				)
-				(hide yes)
-			)
-		)
-		(instances
-			(project "vesc_mms_board"
-				(path "/19c3ad7a-1b7d-4298-9053-cf734bfcea10"
-					(reference "H1")
-					(unit 1)
-				)
-			)
-		)
-	)
 	(symbol
 		(lib_id "Mechanical:MountingHole")
